File: Asymptote_Campitrayhulliander_Plate/Asymptote_Campitrayhulliander_Plate.kicad_pcb (KiCad board)
At the start: 2 copper layers, 251.2 x 85.2 mm, 21 parts

Commit message: asymplate finished?
Parts:
- added REF**: mousebites 1mm, PCM_marbastlib-various:mousebites_1mm, F.Cu at (130.8, 124.5)
- added REF**: mousebites 1mm, PCM_marbastlib-various:mousebites_1mm, B.Cu at (162.6, 124.5)
- added REF**: mousebites 1mm, PCM_marbastlib-various:mousebites_1mm, F.Cu at (251.5, 124.5)
- added REF**: mousebites 1mm, PCM_marbastlib-various:mousebites_1mm, F.Cu at (51.5, 124.5)
- added REF**: mousebites 1mm, PCM_marbastlib-various:mousebites_1mm, F.Cu at (232.4, 124.5)
- added REF**: mousebites 1mm, PCM_marbastlib-various:mousebites_1mm, F.Cu at (58.6, 124.5)
- moved REF** 0.10 mm to (261.3, 65.3)
- moved REF** 0.10 mm to (36.8, 140.8)
- moved REF** 0.10 mm to (261.3, 140.8)
Routing:
- added copper zone on B.Cu, net (none)
- added copper zone on F.Cu, net (none)
Other:
- outline, holes or cut-outs redrawn
- board text added: "JLCJLCJLCJLC"
